File: kicad/SSRU_v3.3/SSRU_v3.3.kicad_pcb (KiCad board)
At the start: 2 copper layers, 95 x 78 mm, 69 parts, among them J2 Conn_01x24, J31 Conn_01x04, J4 AVR-ISP-6, J5 Conn_01x03, SW1 SW_Push, U1 MCP2515-xST, U10 TJA1051T, U12 TJA1051T, U2 ATmega328P-A, U3 LM2904, U4 LM2576S-5, U6 MCP2515-xST, U8 74LVC1G17, Y1 16MHz, Y3 20MHz, Y4 20MHz

Commit message: pudh
Routing:
- net +5V: track 361.3 -> 359.5 mm, vias 13 -> 12
Other:
- board text added: "RBR_SSRU_V3.3 09/02/2026 PCB by Jasmine Lee Code by Jasmine Lee"
- board text removed: "RBR_SSRU_V3.2 23/09/2025 PCB by Nicholas Chan Code by Jasmine Lee"
Changed lines of the file:
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@@
 	)
 	(gr_rect
-		(start 187 78.25)
-		(end 193 79.75)
+		(start 187 79.25)
+		(end 193 80.75)
 		(stroke
 			(width 0.1)
@@
 		(layer "Edge.Cuts")
 	)
-	(gr_text "RBR_SSRU_V3.2\n23/09/2025\nPCB by Nicholas Chan\nCode by Jasmine Lee"
+	(gr_text "RBR_SSRU_V3.3\n09/02/2026\nPCB by Jasmine Lee\nCode by Jasmine Lee"
 		(at 169.75 138.25 0)
 		(layer "F.SilkS")
@@
 	)
 	(segment
-		(start 155 89.7913)
-		(end 153.2156 88.0069)
-		(width 1)
-		(layer "F.Cu")
-		(net 2)
-	)
-	(segment
 		(start 191.7844 97)
 		(end 191.7844 99)
@@
 	)
 	(segment
-		(start 155 97)
-		(end 155 89.7913)
-		(width 1)
-		(layer "F.Cu")
-		(net 2)
-	)
-	(segment
 		(start 194 79)
 		(end 173 79)
@@
 	)
 	(via
-		(at 155 97)
-		(size 1)
-		(drill 0.5)
-		(layers "F.Cu" "B.Cu")
-		(net 2)
-	)
-	(via
 		(at 179.1017 127.4725)
 		(size 0.6)
@@
 	)
 	(segment
-		(start 155 106.6388)
-		(end 155.1456 106.7844)
-		(width 1)
-		(layer "B.Cu")
-		(net 2)
-	)
-	(segment
 		(start 175.79 101.71)
 		(end 179 98.5)
@@
 	)
 	(segment
-		(start 154.9931 96.9931)
-		(end 155 97)
-		(width 0.5)
-		(layer "B.Cu")
-		(net 2)
-	)
-	(segment
 		(start 153.2156 88.0069)
 		(end 155.0069 88.0069)
@@
 	)
 	(segment
-		(start 155 106.6388)
-		(end 155 97)
-		(width 1)
-		(layer "B.Cu")
-		(net 2)
-	)
-	(segment
 		(start 120.125 83.5)
 		(end 121 84.375)
@@
 	)
 	(segment
-		(start 137.6812 96.9931)
-		(end 154.9931 96.9931)
-		(width 0.5)
-		(layer "B.Cu")
-		(net 2)
-	)
-	(segment
 		(start 107.98 88.02)
 		(end 109.975 88.02)
@@
 	)
 	(segment
+		(start 137.6812 96.9931)
+		(end 153.25 96.9931)
+		(width 0.5)
+		(layer "B.Cu")
+		(net 2)
+	)
+	(segment
 		(start 164.62 91)
 		(end 166.6525 93.0325)
@@
 	)
 	(segment
+		(start 153.2156 103.4656)
+		(end 153.2156 88.0069)
+		(width 1)
+		(layer "B.Cu")
+		(net 2)
+	)
+	(segment
 		(start 112.0025 110.8475)
 		(end 109.975 108.82)
@@
 	)
 	(segment
+		(start 155 106.6388)
+		(end 155 105.25)
+		(width 1)
+		(layer "B.Cu")
+		(net 2)
+	)
+	(segment
 		(start 163 91)
 		(end 164.2844 91)
@@
 	)
 	(segment
+		(start 155.1456 106.7844)
+		(end 155 106.6388)
+		(width 1)
+		(layer "B.Cu")
+		(net 2)
+	)
+	(segment
+		(start 155 105.25)
+		(end 153.2156 103.4656)
+		(width 1)
+		(layer "B.Cu")
+		(net 2)
+	)
+	(segment
 		(start 121 84.375)
 		(end 121 87)
@@
 	)
 	(segment
-		(start 125.75 109)
-		(end 132.75 109)
+		(start 178.136218 92.570532)
+		(end 175.815686 90.25)
 		(width 0.25)
 		(layer "F.Cu")
@@
 	)
 	(segment
-		(start 178.136218 92.570532)
-		(end 175.815686 90.25)
+		(start 160 95.5)
+		(end 149.5 95.5)
 		(width 0.25)
 		(layer "F.Cu")
@@
 	)
 	(segment
-		(start 132.75 109)
+		(start 125.75 109)
 		(end 135.5 109)
 		(width 0.25)
@@
 	)
 	(segment
-		(start 149 99.25)
-		(end 149 95.5)
+		(start 149 96)
+		(end 149 99.25)
+		(width 0.25)
+		(layer "F.Cu")
+		(net 7)
+	)
+	(segment
+		(start 149.5 95.5)
+		(end 149 96)
 		(width 0.25)
 		(layer "F.Cu")
@@
 	)
 	(via
-		(at 149 95.5)
+		(at 160 95.5)
 		(size 0.6)
 		(drill 0.3)
@@
 	)
 	(segment
-		(start 125.75 109.5)
+		(start 125.75 112.5)
 		(end 125.75 109)
 		(width 0.25)
@@
 	(segment
 		(start 139.25 105.25)
-		(end 143 105.25)
-		(width 0.25)
-		(layer "B.Cu")
-		(net 7)
-	)
-	(segment
-		(start 143 105.25)
 		(end 148.5 105.25)
 		(width 0.25)
@@
 	)
 	(segment
-		(start 125.75 112.5)
-		(end 125.75 109.5)
-		(width 0.25)
-		(layer "B.Cu")
-		(net 7)
-	)
-	(segment
 		(start 122.285 112.97)
 		(end 122.4675 113.1525)
@@
 	)
 	(segment
-		(start 149 95.5)
-		(end 160 95.5)
-		(width 0.25)
-		(layer "B.Cu")
-		(net 7)
-	)
-	(segment
 		(start 168.75 94.5)
 		(end 169.25 94)
@@
 	(segment
 		(start 189 99.25)
-		(end 190.25 100.5)
-		(width 0.25)
-		(layer "F.Cu")
-		(net 45)
-	)
-	(segment
-		(start 190.25 100.5)
 		(end 191.5 101.75)
 		(width 0.25)
@@
 	)
 	(segment
-		(start 122.665 106.665)
-		(end 135.92919 106.665)
-		(width 0.25)
-		(layer "F.Cu")
-		(net 51)
-	)
-	(segment
 		(start 118.375 105.49)
 		(end 121.49 105.49)
@@
 	)
 	(segment
-		(start 135.92919 106.665)
-		(end 136.30281 106.665)
-		(width 0.25)
-		(layer "F.Cu")
-		(net 51)
-	)
-	(segment
 		(start 158.75 113.5)
 		(end 162.549 117.299)
@@
 	)
 	(segment
-		(start 136.30281 106.665)
+		(start 122.665 106.665)
 		(end 136.415 106.665)
 		(width 0.25)
